Commit message: added gazebo
Signed-off-by: Albert <wensinlor@gmail.com>

File: install/line_follower_description/share/line_follower_description/urdf/common_properties.xacro (robot description, xacro)
@@ -5,5 +5,8 @@
     </material>
     <material name="grey">
-        <color rgba="0.5 0.5 0.5 1"/>
+        <color rgba="0.9 0.9 0.9 1"/>
+    </material>
+    <material name="transparent_grey">
+        <color rgba="0.9 0.9 0.9 0.5"/>
     </material>
     <material name="orange">
@@ -13,11 +16,14 @@
         <color rgba="1.0 1.0 0 1"/>
     </material>
+    <material name="black">
+        <color rgba="0.13 0.13 0.13 1"/>
+    </material>
     <xacro:macro name="box_inertia" params="m l w h xyz rpy">
         <inertial>
             <origin xyz="${xyz}" rpy="${rpy}"/>
             <mass value="${m}"/>
-            <inertia ixx="${(m/12) * (h*h + l*l)}" ixy="0" ixz="0"
-                     iyy="${(m/12) * (w*w + l*l)}" iyz="0"
-                     izz="${(m/12) * (w*w + h*h)}"/>
+            <inertia ixx="${(m/12) * (w*w + h*h)}" ixy="0" ixz="0"
+                     iyy="${(m/12) * (h*h + l*l)}" iyz="0"
+                     izz="${(m/12) * (w*w + l*l)}"/>
         </inertial>
     </xacro:macro>
@@ -27,6 +33,6 @@
             <mass value="${m}"/>
             <inertia ixx="${(m/12) * (3*r*r + h*h)}" ixy="0" ixz="0"
-                     iyy="${(m/12) * (3*r*r + h*h)}" iyz="0"
-                     izz="${(m/2) * (r*r)}"/>
+                     iyy="${(m/2) * (r*r)}" iyz="0"
+                     izz="${(m/12) * (3*r*r + h*h)}"/>
         </inertial>
     </xacro:macro>

File: install/line_follower_description/share/line_follower_description/urdf/line_follower.urdf.xacro (robot description, xacro)
@@ -3,3 +3,4 @@
     <xacro:include filename="common_properties.xacro" />
     <xacro:include filename="mobile_base.xacro" />
+    <xacro:include filename="mobile_base_gazebo.xacro" />
 </robot>

File: install/line_follower_description/share/line_follower_description/urdf/mobile_base.xacro (robot description, xacro)
@@ -4,5 +4,5 @@
     <xacro:property name="base_width" value="0.1"/>
     <xacro:property name="base_height" value="0.003"/>
-    <xacro:property name="wheel_radius" value="0.07"/>
+    <xacro:property name="wheel_radius" value="0.035"/>
     <xacro:property name="wheel_length" value="0.027"/>
     <link name="base_footprint"/>
@@ -13,5 +13,5 @@
             </geometry>
             <origin xyz="0 0 ${base_height / 2.0}" rpy="0 0 0"/>
-            <material name="blue"/>
+            <material name="transparent_grey"/>
         </visual>
         <collision>
@@ -31,5 +31,5 @@
                 </geometry>
                 <origin xyz="0 0 0" rpy="${pi / 2.0} 0 0"/>
-                <material name="grey"/>
+                <material name="black"/>
             </visual>
             <collision>
