Commit message: added line detector node
Signed-off-by: Albert <wensinlor@gmail.com>

File: install/line_follower_description/share/line_follower_description/urdf/camera.xacro (robot description, xacro)
@@ -1,7 +1,7 @@
 <?xml version="1.0"?>
 <robot xmlns:xacro="http://www.ros.org/wiki/xacro">
-    <xacro:property name="camera_length" value="0.0331" />
-    <xacro:property name="camera_width" value="0.014" />
-    <xacro:property name="camera_depth" value="0.001" />
+    <xacro:property name="camera_length" value="0.0001" />
+    <xacro:property name="camera_width" value="0.0001" />
+    <xacro:property name="camera_depth" value="0.0001" />
     <link name="camera_link_0">
         <visual>
@@ -9,5 +9,5 @@
                 <box size="${camera_length} ${camera_width} ${camera_depth}" />
             </geometry>
-            <material name="grey" />
+            <material name="red" />
         </visual>
         <collision>
@@ -16,5 +16,5 @@
             </geometry>
         </collision>
-        <xacro:box_inertia m="0.1" l="${camera_length}" w="${camera_width}" h="${camera_depth}"
+        <xacro:box_inertia m="0.0000000000000000000000000000000001" l="${camera_length}" w="${camera_width}" h="${camera_depth}"
                            xyz="0 0 0" rpy="0 0 0" />
     </link>
@@ -22,7 +22,7 @@
         <parent link="base_link" />
         <child link="camera_link_0" />
-        <origin xyz="${(base_length + camera_depth) / 2.0} 0.036 ${-2*base_height}" rpy="0 ${pi/2} 0" />
+        <origin xyz="${(base_length + camera_depth) / 2.0} 0 0.1" rpy="0 ${pi/2} 0" />
     </joint>
-    <link name="camera_link_1">
+    <!-- <link name="camera_link_1">
         <visual>
             <geometry>
@@ -83,5 +83,5 @@
         <child link="camera_link_3" />
         <origin xyz="${(base_length + camera_depth) / 2.0} -0.036 ${-2*base_height}" rpy="0 ${pi/2} 0" />
-    </joint>
+    </joint> -->
     <link name="camera_link_optical_0">
     </link>
@@ -94,10 +94,7 @@
         <child link="camera_link_optical_0"/>
     </joint>
-    <link name="camera_link_optical_1">
+    <!-- <link name="camera_link_optical_1">
     </link>
     <joint name="camera_optical_joint_1" type="fixed">
-        <!-- these values have to be these values otherwise the gazebo camera
-            image won't be aligned properly with the frame it is supposedly
-            originating from -->
         <origin xyz="0 0 0" rpy="${-pi/2} 0 ${-pi/2}"/>
         <parent link="camera_link_0"/>
@@ -107,7 +104,4 @@
     </link>
     <joint name="camera_optical_joint_2" type="fixed">
-        <!-- these values have to be these values otherwise the gazebo camera
-            image won't be aligned properly with the frame it is supposedly
-            originating from -->
         <origin xyz="0 0 0" rpy="${-pi/2} 0 ${-pi/2}"/>
         <parent link="camera_link_0"/>
@@ -117,11 +111,8 @@
     </link>
     <joint name="camera_optical_joint_3" type="fixed">
-        <!-- these values have to be these values otherwise the gazebo camera
-            image won't be aligned properly with the frame it is supposedly
-            originating from -->
         <origin xyz="0 0 0" rpy="${-pi/2} 0 ${-pi/2}"/>
         <parent link="camera_link_3"/>
         <child link="camera_link_optical_3"/>
-    </joint>
+    </joint> -->
     <gazebo reference="camera_link_0">
         <material>Gazebo/Red</material>
@@ -135,5 +126,5 @@
         </sensor>
     </gazebo>
-    <gazebo reference="camera_link_1">
+    <!-- <gazebo reference="camera_link_1">
         <material>Gazebo/Red</material>
         <sensor name="camera_sensor_1" type="camera">
@@ -167,4 +158,4 @@
             </plugin>
         </sensor>
-    </gazebo>
+    </gazebo> -->
 </robot>

File: install/line_follower_description/share/line_follower_description/urdf/common_properties.xacro (robot description, xacro)
@@ -3,4 +3,7 @@
     <material name="blue">
         <color rgba="0 0 0.5 1"/>
+    </material>
+    <material name="red">
+        <color rgba="0.5 0 0 1"/>
     </material>
     <material name="grey">
