Commit message: added trial-and-error method pid controller
Signed-off-by: Albert <wensinlor@gmail.com>

File: install/line_follower_description/share/line_follower_description/urdf/mobile_base.xacro (robot description, xacro)
@@ -70,5 +70,5 @@
         <parent link="base_link"/>
         <child link="right_wheel_link"/>
-        <origin xyz="${-base_length / 4.0} ${-(base_width + wheel_length) / 2.0} 0" rpy="0 0 0"/>
+        <origin xyz="-0.028 ${-(base_width + wheel_length) / 2.0} 0" rpy="0 0 0"/>
         <axis xyz="0 1 0"/>
     </joint>
@@ -76,5 +76,5 @@
         <parent link="base_link"/>
         <child link="left_wheel_link"/>
-        <origin xyz="${-base_length / 4.0} ${(base_width + wheel_length) / 2.0} 0" rpy="0 0 0"/>
+        <origin xyz="-0.028 ${(base_width + wheel_length) / 2.0} 0" rpy="0 0 0"/>
         <axis xyz="0 1 0"/>
     </joint>
